File: hardware/LEDs/LEDs_10x10/LEDs_10x10.kicad_sch (KiCad schematic)
At the start: 100 parts

Commit message: actualización
Parts:
- added J2: Conn_01x03_Pin, symbol Connector:Conn_01x03_Pin
- added J3: Conn_01x02_Pin, symbol Connector:Conn_01x02_Pin
- added Q2: NPN, Package_TO_SOT_SMD:SOT-223, symbol Simulation_SPICE:NPN
- added R1: 3.3, Resistor_SMD:R_0603_1608Metric, symbol Device:R
- added RV1: R_Potentiometer, symbol Device:R_Potentiometer
- added U1: OPA735, Package_TO_SOT_SMD:TSOT-23-5_HandSoldering, symbol Simulation_SPICE:OPAMP
Connections:
- net Vboost: now also J3.1 (Pin_1)
- net at D10.1 (K), D100.1 (K), D20.1 (K)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: now also Q2.1 (C)
- new net: J2.N, U1.1 (+)
- new net: Q2.3 (E), R1.1, U1.2 (-)
- new net: Q2.2 (B), U1.3
- new net: J2.NC, RV1.2
- new net +3.3V: J2.2 (Pin_2), RV1.1
- new net ADC: J2.1 (Pin_1), J2.NO
- new net Bat: U1.4 (V+)
- new net GND: J2.3 (Pin_3), J3.2 (Pin_2), R1.2, RV1.3, U1.5 (V-)
Other:
- moved on the sheet: D1, D10, D100, D11, D12, D13, D14, D15, D16, D17, D18, D19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

Commit message: pcb
Parts:
- removed J2: Conn_01x03_Pin, symbol Connector:Conn_01x03_Pin
- removed J3: Conn_01x02_Pin, symbol Connector:Conn_01x02_Pin
- removed RV1: R_Potentiometer, symbol Device:R_Potentiometer
- added J1: Conn_01x02_Pin, symbol Connector:Conn_01x02_Pin
- added J4: Conn_01x03_Pin, symbol Connector:Conn_01x03_Pin
Connections:
- net ADC: now also U1.1 (+), J1.1 (Pin_1)
- net Bat: now also J4.3 (Pin_3)
- net GND: now also J1.2 (Pin_2), J4.2 (Pin_2)
- net Vboost: now also J4.1 (Pin_1)

Commit message: editchico
Parts:
- Alimentaciones1: renamed from J4; footprint (none) -> Connector_JST:JST_XH_B3B-XH-A_1x03_P2.50mm_Vertical
- VADC1: renamed from J1; footprint (none) -> Connector_JST:JST_XH_B2B-XH-A_1x02_P2.50mm_Vertical
Changed lines of the file:
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@@
   (symbol (lib_id "Connector:Conn_01x02_Pin") (at 50.8 125.73 0) (unit 1)
     (in_bom yes) (on_board yes) (dnp no) (fields_autoplaced)
-    (property "Reference" "J1" (at 51.435 120.65 0)
+    (property "Reference" "VADC1" (at 51.435 120.65 0)
       (effects (font (size 1.27 1.27)))
     )
@@
       (effects (font (size 1.27 1.27)))
     )
-    (property "Footprint" "" (at 50.8 125.73 0)
+    (property "Footprint" "Connector_JST:JST_XH_B2B-XH-A_1x02_P2.50mm_Vertical" (at 50.8 125.73 0)
       (effects (font (size 1.27 1.27)) hide)
     )
@@
       (project "LEDs_10x10"
         (path "/430e6ebd-258a-4614-8294-6e3f366aedfb"
-          (reference "J1") (unit 1)
+          (reference "VADC1") (unit 1)
         )
       )
@@
   (symbol (lib_id "Connector:Conn_01x03_Pin") (at 102.87 29.845 0) (unit 1)
     (in_bom yes) (on_board yes) (dnp no) (fields_autoplaced)
-    (property "Reference" "J4" (at 103.505 22.225 0)
+    (property "Reference" "Alimentaciones1" (at 103.505 22.86 0)
       (effects (font (size 1.27 1.27)))
     )
-    (property "Value" "Conn_01x03_Pin" (at 103.505 24.765 0)
+    (property "Value" "Conn_01x03_Pin" (at 103.505 25.4 0)
       (effects (font (size 1.27 1.27)))
     )
-    (property "Footprint" "" (at 102.87 29.845 0)
+    (property "Footprint" "Connector_JST:JST_XH_B3B-XH-A_1x03_P2.50mm_Vertical" (at 102.87 29.845 0)
       (effects (font (size 1.27 1.27)) hide)
     )
@@
       (project "LEDs_10x10"
         (path "/430e6ebd-258a-4614-8294-6e3f366aedfb"
-          (reference "J4") (unit 1)
-        )
-      )
+          (reference "Alimentaciones1") (unit 1)
+        )
+      )
