File: hardware/controlador/Transiluminador.kicad_pcb (KiCad board)
At the start: 2 copper layers, 89 parts, among them J1 Conn_01x02_Pin, J10 USB_B_Micro, J11 V_in, J12 V_DD, J13 GND, J14 5V, J15 3.3V, J16 VDL_3V3, J17 VS_3V3, J18 Conn_01x02_Pin, J2 Conn_01x03_Pin, J3 HDR-2x1, J5 Conn_01x03_Pin, J6 Conn_01x05_Pin, J7 HDR-3x1, J8 ST77XX, J9 HDR-3x1, Q1 Q_PMOS_GSD, Q4 Q_Dual_NPN_NPN_BRT_E1B1C2E2B2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, SW2 SW_DIP_x02, SW3 SW_DIP_x02, SW4 SW_DIP_x02, SW5 SW_DIP_x02, U10 ESP32-WROOM-32D, U4 MT3608, U6 AP2112K-3.3, U7 AP2112K-3.3, U8 AP2112K-3.3, U9 CH340C

Commit message: pcb_lista
Parts:
- added G***: LOGO, IoWLabsLogos:IoWLabs_logo_32mm, F.Cu at (153.2, 20.3)
- added G***: LOGO, Imagenes_png:circulo_final_bien, B.Cu at (149.9, 58.4)
- added REF**: OSHW-Logo2_14.6x12mm_SilkScreen, Symbol:OSHW-Logo2_14.6x12mm_SilkScreen, F.Cu at (123.1, 89.6)
- R10, R11, R12, R2, R3, R4, R7, R8, R9: footprint Resistor_SMD:R_0201_0603Metric -> Resistor_SMD:R_0603_1608Metric
- moved D106 150.6 mm to (109.4, 81.3), turned to 180 degrees
- moved 5V1 147.8 mm to (104.6, 71.9)
- moved R13 147.7 mm to (106.2, 77.9)
- moved C8 146.7 mm to (112.1, 78.1), turned to -90 degrees
- moved R10 146.7 mm to (103.6, 82.1), turned to -90 degrees
- moved GND1 142.0 mm to (115.6, 41.8)
- moved R11 138.6 mm to (103.6, 85.6)
- moved D104 129.8 mm to (116.1, 69.9), turned to 0 degrees
- moved U4 119.6 mm to (116.4, 82.0), turned to 0 degrees
- moved F2 117.1 mm to (185.0, 87.6)
- moved L2 115.4 mm to (125.6, 79.2), turned to 90 degrees
- moved V_in1 108.9 mm to (184.2, 69.9), turned to 90 degrees
- moved Alimentacion_12V1 98.7 mm to (169.1, 98.6), turned to 180 degrees
- moved V_Placa_2 97.6 mm to (158.6, 98.6), turned to 180 degrees
- moved L1 89.7 mm to (181.2, 76.2), turned to -90 degrees
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- renumbered J15 to 3.3V1, J14 to 5V1, J3 to Alimentacion_12V1, J6 to Encoder1, J13 to GND1, J8 to PANTALLA1, J18 to VDAC_1, J1 to VDAC_2, J16 to VDL1, J17 to VS1, J12 to V_DD1, J2 to V_Placa_1, J5 to V_Placa_2, J11 to V_in1
Routing:
- net +3.3V: track 0.00 -> 184.4 mm, vias 0 -> 7
- net V_in: track 0.00 -> 107.5 mm
- net +5V: track 0.00 -> 99.3 mm
- net V_DD: track 0.00 -> 95.9 mm
- net V+: track 0.00 -> 72.4 mm, vias 0 -> 2
- net /RESET: track 0.00 -> 59.8 mm, vias 0 -> 3
- net V_12V: track 0.00 -> 54.2 mm, vias 0 -> 1
- net DC: track 0.00 -> 52.4 mm, vias 0 -> 1
- net SPI_MISO: track 0.00 -> 52.4 mm, vias 0 -> 1
- net RES: track 0.00 -> 50.4 mm, vias 0 -> 1
- net SPI_CLK: track 0.00 -> 49.9 mm, vias 0 -> 1
- net CLK_ENCODER: track 0.00 -> 48.3 mm
- net DT_ENCODER: track 0.00 -> 46.4 mm
- net SW_ENCODER: track 0.00 -> 44.6 mm
- net Net-(R14-Pad2): track 0.00 -> 40.0 mm
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- added copper zone on B.Cu, net GND
- added copper zone on F.Cu, net GND
Other:
- board outline added: 100 x 88.5 mm
- board text added: "+"
- board text added: "-"
- board text added: "- +"
- board text added: "12V"
- board text added: "3.3V GND CLK MISO RES DC"
- board text added: "Amaru Rubilar 12-2023 Controlador Transiluminador V1.0"
- board text added: "GND 3.3V SW DT CLK"
- board text added: "Vdd GND Vin"

Commit message: sensorluz
Parts:
- added Senso_Luz1: Conn_01x04_Pin, Connector_JST:JST_XH_B4B-XH-A_1x04_P2.50mm_Vertical, F.Cu at (195.1, 45.1)
- moved R21 7.16 mm to (189.2, 50.6), turned to -90 degrees
- moved SW2 2.74 mm to (191.7, 57.8)
- moved SW3 2.74 mm to (191.7, 54.2)
Routing:
- net scl: track 30.4 -> 54.3 mm, vias 0 -> 1
- net sda: track 30.5 -> 48.0 mm, vias 2 -> 3
- net Net-(R21-Pad2): track 15.7 -> 6.15 mm
- net +3.3V: track 184.4 -> 190.0 mm
- net Net-(R20-Pad2): track 22.4 -> 23.6 mm
- net /RESET: track 59.8 -> 58.9 mm
- net GND: vias 53 -> 52

Commit message: v1.1
Parts:
- removed Alimentacion_12V1: HDR-2x1, Connector_JST:JST_XH_B2B-XH-A_1x02_P2.50mm_Vertical
- removed D104, D105: D_Schottky, Diode_SMD:D_SMA
- removed D106, D107, D108, D109, D111: LED, LED_SMD:LED_0603_1608Metric
- removed the G*** at (153.2, 20.3)
- removed GND1: GND, TestPoint:TestPoint_Loop_D2.50mm_Drill1.0mm_LowProfile
- removed J7, J9: HDR-3x1, Jumper:SolderJumper-3_P1.3mm_Open_RoundedPad1.0x1.5mm_NumberLabels
- removed R12: 4.7k, Resistor_SMD:R_0603_1608Metric
- removed SW5: SW_DIP_x02, IoWLabs:SMD_SWITCH
- removed VDAC_1, VDAC_2: Conn_01x02_Pin, Connector_JST:JST_XH_B2B-XH-A_1x02_P2.50mm_Vertical
- removed VR1: LM2577S-ADJ_NOPB, Transistor:VREG_LM2577S-ADJ_NOPB
- removed V_DD1: V_DD, TestPoint:TestPoint_Loop_D2.50mm_Drill1.0mm_LowProfile
- removed V_in1: V_in, TestPoint:TestPoint_Loop_D2.50mm_Drill1.0mm_LowProfile
- added Alimentacion_12V2: HDR-2x1, Connector_JST:JST_XH_B2B-XH-A_1x02_P2.50mm_Vertical, F.Cu at (194.6, 62.1)
- added C21: 220u, Capacitor_SMD:CP_Elec_10x10.5, F.Cu at (178.6, 94.3)
- added C22: 100n, Capacitor_SMD:C_0603_1608Metric, F.Cu at (121.5, 55.3)
- added C23: 100n, Capacitor_SMD:C_0603_1608Metric, F.Cu at (136.1, 36.1)
- added D3: LED, LED_SMD:LED_0603_1608Metric, F.Cu at (155.3, 47.4)
- added D4: D_Schottky, Diode_SMD:D_SMA, F.Cu at (166.9, 54.0)
- added D5: D_Schottky, Diode_SMD:D_SMA, F.Cu at (188.1, 27.6)
- added D6: LED, LED_SMD:LED_0603_1608Metric, F.Cu at (159.5, 43.8)
- added D7: LED, LED_SMD:LED_0603_1608Metric, F.Cu at (126.4, 28.4)
- added D8: LED, LED_SMD:LED_0603_1608Metric, F.Cu at (126.4, 38.4)
- added D9: LED, LED_SMD:LED_0603_1608Metric, F.Cu at (124.2, 47.9)
- added F3: FUSE, Fuse:Fuse_1206_3216Metric, F.Cu at (189.8, 51.8)
- added G***: LOGO, IoWLabsLogos:IoWLabs_logo, F.Cu at (125.9, 85.6)
- added GND2: GND, TestPoint:TestPoint_Loop_D2.50mm_Drill1.0mm_LowProfile, F.Cu at (182.6, 50.1)
- added Q2: NPN, Package_TO_SOT_SMD:SOT-223-3_TabPin2, F.Cu at (136.8, 83.7)
- added Q3: NPN, Package_TO_SOT_SMD:SOT-223-3_TabPin2, F.Cu at (149.0, 83.7)
- added R18: 5, IoWLabs:TO-263-3 TAB 3, F.Cu at (128.9, 69.2)
- added R26: 5, IoWLabs:TO-263-3 TAB 3, F.Cu at (160.7, 91.7)
- added SW6: ~, IoWLabs:SS-SK12D07VG4-SDDT, F.Cu at (195.0, 51.8)
- added U1: TLC272, Package_SO:SOIC-8_3.9x4.9mm_P1.27mm, F.Cu at (141.9, 73.9)
- added U3: XL6008, Package_TO_SOT_SMD:TO-252-5_TabPin6, F.Cu at (164.2, 74.7)
- C1: value 2200u -> 47u; footprint Capacitor_THT:CP_Radial_D12.5mm_P5.00mm -> Capacitor_SMD:CP_Elec_6.3x7.7
- C10: value 0.1u -> 10u
- C2: value 0.15u -> 1u; footprint Capacitor_SMD:C_0603_1608Metric -> Capacitor_SMD:C_0805_2012Metric
- C3: value 0.1u -> 1u; footprint Capacitor_SMD:C_0603_1608Metric -> Capacitor_SMD:C_0805_2012Metric
- C5: value 10u -> 0.1u
- F2: value FUSE -> Fuse
- L1: value 100u -> 33u; footprint IoWLabs:Inductor_7.5x7.0 -> Inductor_SMD:L_12x12mm_H8mm
- R2: value 12k -> 1k
- R3: value 2.2k -> 11.8k
- R4: value 1k -> 10K
- R7, R8: value 5k -> 10k
- R9: value 4.7k -> 10K
- SW1: value ~ -> SW_Omron_B3FS; footprint IoWLabs:SS-12F23-G040 -> Connector_JST:JST_XH_B2B-XH-A_1x02_P2.50mm_Vertical
- SW4: value SW_DIP_x02 -> SW_Omron_B3FS; footprint IoWLabs:SMD_SWITCH -> Connector_JST:JST_XH_B2B-XH-A_1x02_P2.50mm_Vertical
- U2: value ~ -> MCP4728
- moved Senso_Luz1 93.8 mm to (117.0, 97.0), turned to 0 degrees
- moved PANTALLA1 79.1 mm to (114.8, 89.8), turned to 90 degrees
- moved SW1 78.7 mm to (115.1, 54.3), turned to 90 degrees
- moved 5V1 67.9 mm to (166.9, 45.0), turned to 180 degrees
- moved R10 66.4 mm to (162.8, 52.0), turned to 180 degrees
- moved R13 66.3 mm to (163.1, 43.8), turned to 180 degrees
- moved R11 64.5 mm to (158.7, 52.0), turned to 180 degrees
- moved C8 63.4 mm to (167.9, 48.0), turned to 0 degrees
- moved C6 61.1 mm to (146.1, 68.4)
- moved C7 59.7 mm to (154.1, 71.8), turned to -90 degrees
- moved C10 59.6 mm to (150.8, 71.8), turned to -90 degrees
- moved L2 58.0 mm to (174.6, 48.3), turned to -90 degrees
- moved C5 55.3 mm to (146.1, 64.3), turned to 90 degrees
- moved R4 50.1 mm to (124.5, 51.0)
- moved J10 48.9 mm to (180.4, 16.7), turned to 180 degrees
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Connections:
- C1 pad 1: V_DD -> V_in
- C10 pad 1: Vdac2 -> VS_3V3
- C13 pad 1: /VDL_3V3 -> VDL_3V3
- C16 pad 1: +3.3V -> VDL_3V3
- C2 pad 1: Net-(C2-Pad1) -> Net-(U3-Vin)
- C3 pad 1: V_in -> VCC_H1
- C5 pad 1: +3.3V -> Vdac1
- C6 pad 1: +3.3V -> Vdac2
- C7 pad 1: Vdac1 -> VS_3V3
- D2 pad 1: V_DD -> VCC_H1
- F1 pad 1: V_in -> Net-(J10-VBUS)
- F2 pad 1: V_in -> Net-(U3-Vin)
- F2 pad 2: Net-(SW1-B) -> V_in
- J10 pad 1: V_in -> Net-(J10-VBUS)
- L1 pad 1: V_in -> Net-(U3-Vin)
- Q1 pad 3: V_12V -> V_in
- R16 pad 1: /VDL_3V3 -> VDL_3V3
- R2 pad 1: V_DD -> Net-(D1-A)
- R2 pad 2: Net-(VR1-FEEDBACK) -> V_in
- R22 pad 1: +3.3V -> VDL_3V3
- R24 pad 1: +3.3V -> VDL_3V3
- R3 pad 1: Net-(VR1-COMP) -> Net-(U3-FB)
- R3 pad 2: Net-(C2-Pad1) -> VCC_H1
- R4 pad 1: Net-(VR1-FEEDBACK) -> VDL_3V3
- R4 pad 2: GND -> UP
- R5 pad 1: V_in -> GND
- R5 pad 2: Net-(D1-A) -> Net-(U3-FB)
- R7 pad 1: +3.3V -> VS_3V3
- R8 pad 1: +3.3V -> VS_3V3
- R9 pad 1: Net-(U2-A1) -> VDL_3V3
- R9 pad 2: GND -> DOWN
- SW1 pad 1: V_12V -> GND
- SW1 pad 2: Net-(SW1-B) -> Net-(R1-Pad2)
- SW4 pad 2: GND -> Net-(R14-Pad2)
- U2 pad 1: +3.3V -> VS_3V3
- U2 pad 10: sda -> GND
- U2 pad 2: Net-(U2-A0) -> scl
- U2 pad 3: unconnected-(U2-Vref-Pad3) -> sda
- U2 pad 4: Vdac1 -> unconnected-(U2-~{LDAC}-Pad4)
- U2 pad 5: Vdac2 -> unconnected-(U2-RDY/~{BSY}-Pad5)
- U2 pad 6: unconnected-(U2-LAT/HVC-Pad6) -> Vdac1
- U2 pad 7: GND -> Vdac2
- U2 pad 8: Net-(U2-A1) -> unconnected-(U2-VOUTC-Pad8)
- U2 pad 9: scl -> unconnected-(U2-VOUTD-Pad9)
- U7 pad 3: /EN_VDL_S -> +5V
- U7 pad 5: /VDL_3V3 -> VDL_3V3
- U8 pad 3: /EN_VS_S -> +5V
- U9 pad 16: +3.3V -> VDL_3V3
- U9 pad 4: +3.3V -> VDL_3V3
- VDL1 pad 1: /VDL_3V3 -> VDL_3V3
- V_Placa_1 pad 1: V_in -> GND
- V_Placa_1 pad 2: GND -> I_LED_1
- V_Placa_1 pad 3: V_DD -> VCC_H1
- V_Placa_2 pad 1: V_in -> GND
- V_Placa_2 pad 2: GND -> I_LED_2
- V_Placa_2 pad 3: V_DD -> VCC_H1
Routing:
- net VDL_3V3: track 0.00 -> 118.4 mm, vias 0 -> 3
- net V_DD: track 95.9 -> 0.00 mm
- net VCC_H1: track 0.00 -> 73.9 mm
- net VS_3V3: track 35.3 -> 106.1 mm, vias 0 -> 3
- net +3.3V: track 190.0 -> 120.5 mm, vias 7 -> 0
- net scl: track 54.3 -> 111.6 mm, vias 1 -> 4
- net V_12V: track 54.2 -> 11.1 mm, vias 1 -> 0
- net sda: track 48.0 -> 90.0 mm
- net Net-(Q2-B): track 0.00 -> 39.9 mm, vias 0 -> 2
- net Net-(Q3-E): track 0.00 -> 39.5 mm, vias 0 -> 2
- net UP: track 5.94 -> 35.2 mm, vias 0 -> 2
- net Net-(U3-FB): track 0.00 -> 28.0 mm
- net Net-(R14-Pad2): track 40.0 -> 12.5 mm, vias 0 -> 1
- net Net-(U3-Vin): track 0.00 -> 23.4 mm
- net SPI_CLK: track 49.9 -> 72.8 mm, vias 1 -> 3
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Other:
- board size 100 x 88.5 mm -> 90.3 x 88.5 mm
- board text added: "Lab Teclibre"
- board text added: "Transiluminador"
- board text added: "Transiluminador V1.1 Amaru Rubilar 1-2024"
- board text removed: "+"
- board text removed: "-"
- board text removed: "- +"
- board text removed: "12V"
- board text removed: "3.3V GND CLK MISO RES DC"
- board text removed: "Amaru Rubilar 12-2023 Controlador Transiluminador V1.0"
- board text removed: "GND 3.3V SW DT CLK"
- board text removed: "Vdd GND Vin"

Commit message: esquinas
Routing:
- net GND: track 19.4 -> 35.8 mm, vias 38 -> 39
- net +3.3V: track 120.5 -> 126.3 mm
- net VCC_H1: track 73.9 -> 75.7 mm
- net +5V: track 117.8 -> 116.2 mm
- net V_in: track 87.3 -> 88.6 mm
- net sda: track 90.0 -> 91.1 mm
- net V+: track 63.4 -> 62.9 mm
Other:
- outline, holes or cut-outs redrawn

Commit message: minimos
Parts:
- R18, R26: value 5 -> 3.3
- moved G*** 1.68 mm to (154.1, 60.0)
- moved R11 1.24 mm to (159.6, 52.8), turned to -90 degrees
- moved C18 1.02 mm to (181.1, 44.0), turned to -90 degrees
Connections:
- Q2 pad 3: Net-(Q2-B) -> Net-(Q2-E)
- R18 pad 2: Net-(Q2-B) -> Net-(Q2-E)
- U1 pad 2: Net-(Q2-B) -> Net-(Q2-E)
Routing:
- net Net-(Q2-E): track 0.00 -> 24.2 mm
- net Net-(Q2-B): track 39.9 -> 18.1 mm
- net /RESET: track 65.6 -> 62.0 mm
- net GND: track 35.8 -> 37.6 mm, vias 39 -> 40
- net Net-(D3-A): track 0.00 -> 1.51 mm
- net /FB_5V: track 7.18 -> 8.05 mm

Commit message: cambios_pcb
Parts:
- moved G*** 67.7 mm to (132.8, 18.2)
Other:
- board text added: "DC RES MISO CLK GND 3V3"
- board text added: "DOWN"
- board text added: "GND 3V3 SW DT CLK"
- board text added: "GND I_LED VCC"
- board text added: "SCL SDA GND 3V3"
- board text added: "UP"
- board text added: "V+"
- board text added: "V-"
- board text removed: "Lab Teclibre"

Commit message: actualizacion_loadsharing
Parts:
- moved R6 14.8 mm to (196.0, 29.6)
- moved Q1 6.11 mm to (187.7, 27.6), turned to 180 degrees
- moved D5 4.68 mm to (192.7, 26.8), turned to -90 degrees
- moved F1 2.76 mm to (181.7, 26.0), turned to -90 degrees
Connections:
- D5 pad 2: V_USB -> V_in
- Q1 pad 1: V_USB -> V_in
- Q1 pad 3: V_in -> V_USB
- R6 pad 1: V_USB -> V_in
Routing:
- net V_USB: track 14.8 -> 6.85 mm
- net V_in: track 88.6 -> 94.6 mm
- net GND: track 37.6 -> 42.5 mm, vias 40 -> 42
- net V+: track 62.9 -> 66.9 mm
- net Net-(J10-VBUS): track 5.50 -> 6.49 mm
