File: hardware/controlador/Transiluminador.kicad_sch (KiCad schematic)
At the start: 84 parts, among them J1 Conn_01x01_Pin, J10 USB_B_Micro, J11 HDR-2x1, J12 Conn_01x02, J3 HDR-2x1, J7 HDR-3x1, J9 HDR-3x1, Q1 Q_PMOS_GSD, Q2 NPN, Q4 Q_Dual_NPN_NPN_BRT_E1B1C2E2B2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, SW2 SW_DIP_x02, SW3 SW_DIP_x02, U1 ${SIM.PARAMS}, U10 ESP32-WROOM-32D, U11 RV-8803, U4 MT3608, U6 AP2112K-3.3, U7 AP2112K-3.3, U8 AP2112K-3.3, U9 CH340C

Commit message: actualización
Parts:
- removed J1: Conn_01x01_Pin, Connector_PinHeader_1.00mm:PinHeader_1x01_P1.00mm_Horizontal, symbol Connector:Conn_01x01_Pin
- added C10, C6, C7: 0.1u, Capacitor_SMD:C_0603_1608Metric, symbol IoWLabs:C
- added C5: 10u, Capacitor_SMD:C_0603_1608Metric, symbol IoWLabs:C
- added J2: XLR3_Switched, symbol Connector_Audio:XLR3_Switched
- added R12, R9: 4.7k, symbol Device:R
- added R7, R8: 5k, symbol Device:R
- added RV1: R_Potentiometer, symbol Device:R_Potentiometer
- added U2: ~, Package_SO:MSOP-10_3x3mm_P0.5mm, symbol IoWLabs:MCP47CB
- C3: footprint (none) -> Capacitor_SMD:C_0603_1608Metric
Connections:
- net +5V: now also RV1.1
- net GND: now also C10.2, C5.2, C6.2, C7.2, R12.2, R9.2, RV1.3, U2.7 (Vss)
- net scl: now also R8.2, U2.9 (SCL)
- net sda: now also R7.2, U2.10 (SDA)
- net at U1.1 (+): now also J2.N
- new net: C5.1, C6.1, R7.1, R8.1, U2.1 (Vdd)
- new net: R12.1, U2.2 (A0)
- new net: R9.1, U2.8 (A1)
- new net: J2.NC, RV1.2
- new net Vdac1: C7.1, J2.NO, U2.4 (Vout0)
- new net Vdac2: C10.1, U2.5 (Vout1)
Other:
- note added: "I2C DAC 2 Channels"
- note removed: "Sensors and signal conditioning"
- moved on the sheet: Q2, R1, U1

Commit message: actualización
Parts:
- removed BT2: Battery_Cell, Battery:BatteryHolder_Keystone_3000_1x12mm, symbol Device:Battery_Cell
- removed C21: 10u, Capacitor_SMD:C_0805_2012Metric, symbol IoWLabs:C
- removed C22: 10n, Capacitor_SMD:C_0603_1608Metric, symbol IoWLabs:C
- removed C23: 100n, Capacitor_SMD:C_0603_1608Metric, symbol IoWLabs:C
- removed D101: D_Zener, symbol Device:D_Zener
- removed D112: BAS70-05, Package_TO_SOT_SMD:SOT-23, symbol IoWLabs:BAS70-05
- removed J11: HDR-2x1, Connector_PinHeader_2.54mm:PinHeader_1x02_P2.54mm_Vertical, symbol IoWLabsConnectors:HDR-2x1
- removed J12: Conn_01x02, Jumper:SolderJumper-2_P1.3mm_Open_RoundedPad1.0x1.5mm, symbol Connector_Generic:Conn_01x02
- removed J13: ~, IoWLabsConnectors:microSD_push_push, symbol IoWLabsConnectors:microsd_push_push
- removed J2: XLR3_Switched, symbol Connector_Audio:XLR3_Switched
- removed Q2: NPN, Transistor:SOT-457, symbol Simulation_SPICE:NPN
- removed R1: 5, Resistor_SMD:R_0603_1608Metric, symbol Device:R
- removed R26, R27, R28, R29, R30: 3.3k, Resistor_SMD:R_0603_1608Metric, symbol IoWLabs:RES
- removed R31, R32: 100k, Resistor_SMD:R_0603_1608Metric, symbol IoWLabs:RES
- removed R33, R34: 2.2k, Resistor_SMD:R_0603_1608Metric, symbol IoWLabs:RES
- removed RV1: R_Potentiometer, symbol Device:R_Potentiometer
- removed U1: ${SIM.PARAMS}, symbol Simulation_SPICE:OPAMP
- removed U11: RV-8803, IoWLabs:SON-8, symbol IoWLabs:RV-8803
- added D2: D_Schottky, Diode_SMD:D_SMA, symbol Device:D_Schottky
- added F2: FUSE, Fuse:Fuse_1206_3216Metric, symbol IoWLabs:FUSE
- added J1, J2, J4, J5: Conn_01x03_Pin, Connector_JST:JST_XH_B3B-XH-A_1x03_P2.50mm_Vertical, symbol Connector:Conn_01x03_Pin
- added J11: V_in, symbol Connector:Conn_01x01_Pin
- added J12: V_DD, symbol Connector:Conn_01x01_Pin
- added J13: GND, symbol Connector:Conn_01x01_Pin
- added J14: 5V, symbol Connector:Conn_01x01_Pin
- added J15: 3.3V, symbol Connector:Conn_01x01_Pin
- added J16: VDL_3V3, symbol Connector:Conn_01x01_Pin
- added J17: VS_3V3, symbol Connector:Conn_01x01_Pin
- added J6: Conn_01x05_Pin, Connector_JST:JST_XH_B5B-XH-A_1x05_P2.50mm_Vertical, symbol Connector:Conn_01x05_Pin
- added J8: ST77XX, Connector_JST:JST_XH_B6B-XH-A_1x06_P2.50mm_Vertical, symbol Connector:Conn_01x06_Pin
- C1: footprint (none) -> Capacitor_THT:CP_Radial_D12.5mm_P5.00mm
- C2: footprint (none) -> Capacitor_SMD:C_0603_1608Metric
- J3: footprint (none) -> Connector_JST:JST_XH_B2B-XH-A_1x02_P2.50mm_Vertical
- L1: footprint (none) -> IoWLabs:Inductor_7.5x7.0
- R10, R11: footprint Resistor_SMD:R_0603_1608Metric -> Resistor_SMD:R_0201_0603Metric
- R12, R7, R8, R9: footprint (none) -> Resistor_SMD:R_0201_0603Metric
Connections:
- net +3V3: now also C5.1, C6.1, R7.1, R8.1, U2.1 (Vdd), J1.2 (Pin_2), J15.1 (Pin_1), J4.2 (Pin_2), J8.1 (Pin_1)
- net +5V: now also J14.1 (Pin_1)
- net GND: now also J1.1 (Pin_1), J13.1 (Pin_1), J2.2 (Pin_2), J4.1 (Pin_1), J5.2 (Pin_2), J6.5 (Pin_5), J8.2 (Pin_2)
- net VDL_3V3: now also J16.1 (Pin_1)
- net VS_3V3: now also J17.1 (Pin_1), J6.4 (Pin_4)
- net V_DD: now also D2.1 (K), J12.1 (Pin_1), J2.3 (Pin_3), J5.3 (Pin_3)
- net V_in: now also F2.1, J11.1 (Pin_1), J2.1 (Pin_1), J5.1 (Pin_1); no longer SW1.2 (B)
- net Vdac1: now also J1.3 (Pin_3)
- net Vdac2: now also J4.3 (Pin_3)
- net at L1.2, VR1.4 (SWITCH): now also D2.2 (A)
- net CLK_ENCODER: now reaches U10.10 (IO25)
- net CLK_ENCODER: now also J6.1 (Pin_1)
- net DT_ENCODER: now reaches U10.11 (IO26)
- net DT_ENCODER: now also J6.2 (Pin_2)
- net SW_ENCODER: now reaches U10.12 (IO27)
- net SW_ENCODER: now also J6.3 (Pin_3)
- net DC: now reaches U10.23 (IO15)
- net DC: now also J8.6 (Pin_6)
- net RES: now reaches U10.28 (IO17)
- net RES: now also J8.5 (Pin_5)
- net spi_clk renamed SPI_CLK
- net SPI_CLK: now also J8.3 (Pin_3)
- net spi_miso renamed SPI_MISO
- net SPI_MISO: now also J8.4 (Pin_4)
- new net: F2.2, SW1.2 (B)
- no-connect marks 9 -> 6
Other:
- note added: "Conector encoder"
- note added: "Conectores"
- note added: "Pantalla ST7789/ST7735"
- note added: "Placa Led 1"
- note added: "Placa Led 2"
- note removed: "Current loop"
- note removed: "Datalogger RTC"
- note removed: "I2C addres: 0x32"
- note removed: "MICROSD READER"
- note removed: "current loop supply"
- moved on the sheet: C10, C5, C6, C7, R12, R7, R8, R9, U2

Commit message: pcb
Parts:
- removed J1, J4: Conn_01x03_Pin, Connector_JST:JST_XH_B3B-XH-A_1x03_P2.50mm_Vertical, symbol Connector:Conn_01x03_Pin
- added J1, J18: Conn_01x02_Pin, Connector_JST:JST_XH_B2B-XH-A_1x02_P2.50mm_Vertical, symbol Connector:Conn_01x02_Pin
- added R1, R14: 200, Resistor_SMD:R_0603_1608Metric, symbol IoWLabs:RES
- added SW4, SW5: SW_DIP_x02, IoWLabs:SMD_SWITCH, symbol Switch:SW_DIP_x02
- J11, J12, J13, J14, J15, J16, J17: footprint (none) -> TestPoint:TestPoint_Loop_D2.50mm_Drill1.0mm_LowProfile
Connections:
- net GND: now also J1.1 (Pin_1), J18.1 (Pin_1), SW4.1, SW4.2, SW5.1, SW5.2
- net Vdac1: now also J18.2 (Pin_2)
- net Vdac2: now also J1.2 (Pin_2)
- net UP: now reaches U10.8 (IO32)
- net UP: now also R1.1
- net DOWN: now reaches U10.9 (IO33)
- net DOWN: now also R14.1
- new net: R1.2, SW4.3, SW4.4
- new net: R14.2, SW5.3, SW5.4
Other:
- note added: "Botones Selección Manual"

Commit message: pcb_lista
Parts:
- R10, R11, R12, R2, R3, R4, R7, R8, R9: footprint Resistor_SMD:R_0201_0603Metric -> Resistor_SMD:R_0603_1608Metric
- renumbered J15 to 3.3V1, J14 to 5V1, J3 to Alimentacion_12V1, J6 to Encoder1, J13 to GND1, J8 to PANTALLA1, J18 to VDAC_1, J1 to VDAC_2, J16 to VDL1, J17 to VS1, J12 to V_DD1, J2 to V_Placa_1, J5 to V_Placa_2, J11 to V_in1

Commit message: sensorluz
Parts:
- added Senso_Luz1: Conn_01x04_Pin, Connector_JST:JST_XH_B4B-XH-A_1x04_P2.50mm_Vertical, symbol Connector:Conn_01x04_Pin
Connections:
- net +3V3: now also Senso_Luz1.4 (Pin_4)
- net GND: now also Senso_Luz1.3 (Pin_3)
- net scl: now also Senso_Luz1.1 (Pin_1)
- net sda: now also Senso_Luz1.2 (Pin_2)
Other:
- note added: "Sensor de Luz"
Changed lines of the file:
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@@
     (stroke (width 0) (type default))
   )
+  (wire (pts (xy 485.14 80.645) (xy 488.315 80.645))
+    (stroke (width 0) (type default))
+  )
   (wire (pts (xy 187.325 109.855) (xy 189.865 109.855))
     (stroke (width 0) (type default))
@@
     (stroke (width 0) (type default))
   )
+  (wire (pts (xy 485.14 73.025) (xy 488.315 73.025))
+    (stroke (width 0) (type default))
+  )
   (wire (pts (xy 478.79 33.655) (xy 474.98 33.655))
     (stroke (width 0) (type default))
@@
     (stroke (width 0) (type default))
   )
+  (wire (pts (xy 485.14 75.565) (xy 488.315 75.565))
+    (stroke (width 0) (type default))
+  )
   (wire (pts (xy 156.845 121.92) (xy 156.845 120.65))
     (stroke (width 0) (type default))
@@
     (stroke (width 0) (type default))
   )
+  (wire (pts (xy 485.14 78.105) (xy 488.315 78.105))
+    (stroke (width 0) (type default))
+  )
   (wire (pts (xy 212.725 123.825) (xy 212.725 122.555))
     (stroke (width 0) (type default))
@@
     (fill (type none))
   )
+  (rectangle (start 466.725 62.865) (end 513.08 88.265)
+    (stroke (width 0) (type default))
+    (fill (type none))
+  )
   (rectangle (start 129.54 90.17) (end 240.03 160.02)
     (stroke (width 0) (type default))
@@
     (effects (font (size 2.9972 2.9972) (thickness 0.5994) bold) (justify left bottom))
   )
+  (text "Sensor de Luz" (at 474.345 68.58 0)
+    (effects (font (size 2.9972 2.9972) (thickness 0.5994) bold) (justify left bottom))
+  )
   (text "TRANSILLUMINATOR CONTROLLER" (at 801.37 201.295 0)
     (effects (font (size 2.0066 2.0066)) (justify left bottom))
@@
     )
   )
+  (global_label "+3.3V" (shape input) (at 485.14 73.025 180) (fields_autoplaced)
+    (effects (font (size 1.27 1.27)) (justify right))
+    (property "Intersheetrefs" "${INTERSHEET_REFS}" (at 476.47 73.025 0)
+      (effects (font (size 1.27 1.27)) (justify right) hide)
+    )
+  )
   (global_label "+5V" (shape input) (at 93.98 135.89 0) (fields_autoplaced)
     (effects (font (size 1.27 1.27)) (justify left))
@@
     )
   )
+  (global_label "GND" (shape input) (at 485.14 75.565 180) (fields_autoplaced)
+    (effects (font (size 1.27 1.27)) (justify right))
+    (property "Intersheetrefs" "${INTERSHEET_REFS}" (at 478.2843 75.565 0)
+      (effects (font (size 1.27 1.27)) (justify right) hide)
+    )
+  )
   (global_label "V_DD" (shape input) (at 419.735 46.355 180) (fields_autoplaced)
     (effects (font (size 1.27 1.27)) (justify right))
@@
     )
   )
+  (global_label "scl" (shape input) (at 485.14 80.645 180) (fields_autoplaced)
+    (effects (font (size 1.27 1.27)) (justify right))
+    (property "Intersheetrefs" "${INTERSHEET_REFS}" (at 479.3729 80.645 0)
+      (effects (font (size 1.27 1.27)) (justify right) hide)
+    )
+  )
   (global_label "V_in" (shape input) (at 26.035 50.8 180) (fields_autoplaced)
     (effects (font (size 1.27 1.27)) (justify right))
@@
     )
   )
+  (global_label "sda" (shape input) (at 485.14 78.105 180) (fields_autoplaced)
+    (effects (font (size 1.27 1.27)) (justify right))
+    (property "Intersheetrefs" "${INTERSHEET_REFS}" (at 478.8287 78.105 0)
+      (effects (font (size 1.27 1.27)) (justify right) hide)
+    )
+  )
   (global_label "RES" (shape input) (at 427.355 119.38 0) (fields_autoplaced)
     (effects (font (size 1.27 1.27)) (justify left))
@@
         )
       )
+    )
+  )
+  (symbol (lib_id "Connector:Conn_01x04_Pin") (at 493.395 78.105 180) (unit 1)
+    (in_bom yes) (on_board yes) (dnp no) (fields_autoplaced)
+    (property "Reference" "Senso_Luz1" (at 495.3 75.565 0)
+      (effects (font (size 1.27 1.27)) (justify right))
+    )
+    (property "Value" "Conn_01x04_Pin" (at 495.3 78.105 0)
+      (effects (font (size 1.27 1.27)) (justify right))
+    )
+    (property "Footprint" "Connector_JST:JST_XH_B4B-XH-A_1x04_P2.50mm_Vertical" (at 493.395 78.105 0)
+      (effects (font (size 1.27 1.27)) hide)
+    )
+    (property "Datasheet" "~" (at 493.395 78.105 0)
+      (effects (font (size 1.27 1.27)) hide)
+    )
+    (pin "1")
+    (pin "4")
+    (pin "2")
+    (pin "3")
+    (instances
+      (project "Transiluminador"
+        (path "/3bccb558-cfc1-47b0-87de-a688fdd981c6"
+          (reference "Senso_Luz1") (unit 1)
+        )
+      )

Commit message: v1.1
Parts:
- removed Alimentacion_12V1: HDR-2x1, Connector_JST:JST_XH_B2B-XH-A_1x02_P2.50mm_Vertical, symbol IoWLabsConnectors:HDR-2x1
- removed C2: 0.15u, Capacitor_SMD:C_0603_1608Metric, symbol Device:C_Polarized
- removed C3: 0.1u, Capacitor_SMD:C_0603_1608Metric, symbol Device:C_Polarized
- removed F2: FUSE, Fuse:Fuse_1206_3216Metric, symbol IoWLabs:FUSE
- removed GND1: GND, TestPoint:TestPoint_Loop_D2.50mm_Drill1.0mm_LowProfile, symbol Connector:Conn_01x01_Pin
- removed J7, J9: HDR-3x1, Jumper:SolderJumper-3_P1.3mm_Open_RoundedPad1.0x1.5mm_NumberLabels, symbol IoWLabsConnectors:HDR-3x1
- removed R12, R9: 4.7k, Resistor_SMD:R_0603_1608Metric, symbol Device:R
- removed R4: 1k, Resistor_SMD:R_0603_1608Metric, symbol Device:R
- removed R5: 1k, Resistor_SMD:R_0603_1608Metric, symbol IoWLabs:RES
- removed SW1: ~, IoWLabs:SS-12F23-G040, symbol IoWLabs:SW_SPDT_GND
- removed SW4, SW5: SW_DIP_x02, IoWLabs:SMD_SWITCH, symbol Switch:SW_DIP_x02
- removed U2: ~, Package_SO:MSOP-10_3x3mm_P0.5mm, symbol IoWLabs:MCP47CB
- removed VDAC_1, VDAC_2: Conn_01x02_Pin, Connector_JST:JST_XH_B2B-XH-A_1x02_P2.50mm_Vertical, symbol Connector:Conn_01x02_Pin
- removed VR1: LM2577S-ADJ_NOPB, Transistor:VREG_LM2577S-ADJ_NOPB, symbol Personal:LM2577S-ADJ_NOPB
- removed V_DD1: V_DD, TestPoint:TestPoint_Loop_D2.50mm_Drill1.0mm_LowProfile, symbol Connector:Conn_01x01_Pin
- removed V_in1: V_in, TestPoint:TestPoint_Loop_D2.50mm_Drill1.0mm_LowProfile, symbol Connector:Conn_01x01_Pin
- added Alimentacion_12V2: HDR-2x1, Connector_JST:JST_XH_B2B-XH-A_1x02_P2.50mm_Vertical, symbol IoWLabsConnectors:HDR-2x1
- added C2, C3: 1u, Capacitor_SMD:C_0805_2012Metric, symbol Device:C
- added C21: 220u, Capacitor_SMD:CP_Elec_10x10.5, symbol Device:C_Polarized
- added C22, C23: 100n, Capacitor_SMD:C_0603_1608Metric, symbol IoWLabs:C
- added F2: Fuse, Fuse:Fuse_1206_3216Metric, symbol Device:Fuse
- added F3: FUSE, Fuse:Fuse_1206_3216Metric, symbol IoWLabs:FUSE
- added GND2: GND, TestPoint:TestPoint_Loop_D2.50mm_Drill1.0mm_LowProfile, symbol Connector:Conn_01x01_Pin
- added Q2, Q3: NPN, Package_TO_SOT_SMD:SOT-223-3_TabPin2, symbol Simulation_SPICE:NPN
- added R18, R26: 5, IoWLabs:TO-263-3 TAB 3, symbol Device:R
- added R4, R9: 10K, Resistor_SMD:R_0603_1608Metric, symbol IoWLabs:RES
- added R5: 1k, Resistor_SMD:R_0603_1608Metric, symbol Device:R
- added SW1, SW4: SW_Omron_B3FS, Connector_JST:JST_XH_B2B-XH-A_1x02_P2.50mm_Vertical, symbol Switch:SW_Omron_B3FS
- added SW6: ~, IoWLabs:SS-SK12D07VG4-SDDT, symbol IoWLabs:SW_SPDT_GND
- added U1: TLC272, Package_SO:SOIC-8_3.9x4.9mm_P1.27mm, symbol Amplifier_Operational:TLC272
- added U2: MCP4728, Package_SO:MSOP-10_3x3mm_P0.5mm, symbol Analog_DAC:MCP4728
- added U3: XL6008, Package_TO_SOT_SMD:TO-252-5_TabPin6, symbol IoWLabs:XL6008
- C1: value 2200u -> 47u; footprint Capacitor_THT:CP_Radial_D12.5mm_P5.00mm -> Capacitor_SMD:CP_Elec_6.3x7.7
- C10: value 0.1u -> 10u
- C5: value 10u -> 0.1u
- D1: Color Blue -> (none)
- L1: value 100u -> 33u; footprint IoWLabs:Inductor_7.5x7.0 -> Inductor_SMD:L_12x12mm_H8mm
- R2: value 12k -> 1k
- R3: value 2.2k -> 11.8k
- R7, R8: value 5k -> 10k
- renumbered D111 to D3, D104 to D4, D105 to D5, D106 to D6, D107 to D7, D108 to D8, D109 to D9
Connections:
- net EN_VDL_S is gone; now on net +5V: U7.3 (EN)
- net EN_VS_S is gone; now on net +5V: U8.3 (EN)
- net +3V3: no longer C16.1, C5.1, C6.1, R22.1, R24.1, R7.1, R8.1, U9.16 (VCC), U9.4 (V3)
- net DOWN: now also C23.1, R9.2
- net GND: now also V_Placa_1.1 (Pin_1), V_Placa_2.1 (Pin_1), Alimentacion_12V2.2, C2.2, C21.2, C22.2, C23.2, C3.2, GND2.1 (Pin_1), R18.1, R26.1, R5.1, SW1.1, SW4.1, SW6.3 (C), SW6.4, U1.4 (V-), U2.10 (VSS), U3.1 (GND); no longer V_Placa_1.2 (Pin_2), V_Placa_2.2 (Pin_2)
- net UP: now also C22.1, R4.2
- net VDL_3V3: now also C16.1, R22.1, R24.1, U9.16 (VCC), U9.4 (V3), R4.1, R9.1
- net VS_3V3: now also C10.1, C7.1, R7.1, R8.1, U2.1 (VDD)
- net V_12V: now also Alimentacion_12V2.1, SW6.1 (A); no longer Q1.3 (D)
- net V_in: now also C1.1, Q1.3 (D), R2.2, F2.2, F3.1, U1.8 (V+); no longer F1.1, J10.1 (VBUS), L1.1, V_Placa_1.1 (Pin_1), V_Placa_2.1 (Pin_1)
- net Vdac1: now also C5.1, U1.3 (+), U2.6 (VOUTA); no longer C7.1
- net Vdac2: now also C6.1, U1.5 (+), U2.7 (VOUTB); no longer C10.1
- net scl: now also U2.2 (SCL)
- net sda: now also U2.3 (SDA)
- net at R1.2: now also SW1.2
- net VCC_H1: now reaches R3.2
- net VCC_H1: now also D2.1 (K), V_Placa_1.3 (Pin_3), V_Placa_2.3 (Pin_3), C21.1, C3.1
- net at D2.2 (A), L1.2: now also U3.3 (SW), U3.6 (TAB)
- net at D1.2 (A): now also R2.1
- net at R14.2: now also SW4.2
- net at R3.1: now also R5.2, U3.5 (FB)
- removed net V_DD: C1.1, D2.1 (K), R2.1, V_Placa_1.3 (Pin_3), V_Placa_2.3 (Pin_3)
- new net: Q3.2 (B), U1.7
- new net: Q3.3 (E), R26.2, U1.6 (-)
- new net: F1.1, J10.1 (VBUS)
- new net: Q2.2 (B), U1.1
- new net: Q2.3 (E), R18.2, U1.2 (-)
- new net: F3.2, SW6.2 (B)
- new net: C2.1, F2.1, L1.1, U3.4 (Vin)
- new net 3.3V: U3.2 (EN)
- new net I_LED_1: Q2.1 (C), V_Placa_1.2 (Pin_2)
- new net I_LED_2: Q3.1 (C), V_Placa_2.2 (Pin_2)
Other:
- note added: "Control de corriente"
- note added: "Fuente de poder"
- note added: "I2C DAC 4 Channels"
- note added: "Interruptor de encendido"
- note added: "Up Voltaqe"
- note removed: "I2C DAC 2 Channels"
- note removed: "POWER IN"
- moved on the sheet: R1, R14, Senso_Luz1, V_Placa_1, V_Placa_2

Commit message: minimos
Parts:
- R18, R26: value 5 -> 3.3
Changed lines of the file:
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@@
       (effects (font (size 1.27 1.27)) (justify right))
     )
-    (property "Value" "5" (at 562.61 148.59 0)
+    (property "Value" "3.3" (at 562.61 148.59 0)
       (effects (font (size 1.27 1.27)) (justify right))
     )
@@
       (effects (font (size 1.27 1.27)) (justify right))
     )
-    (property "Value" "5" (at 511.81 147.955 0)
+    (property "Value" "3.3" (at 511.81 147.955 0)
       (effects (font (size 1.27 1.27)) (justify right))
     )

Commit message: actualizacion_loadsharing
Connections:
- net V_USB: now also Q1.3 (D); no longer D5.2 (A), Q1.1 (G), R6.1
- net V_in: now also D5.2 (A), Q1.1 (G), R6.1; no longer Q1.3 (D)
