File: electronics/controlador/Transiluminador.kicad_pcb (KiCad board)
At the start: 2 copper layers, 90.3 x 88.5 mm, 95 parts, among them J10 USB_B_Micro, Q1 Q_PMOS_GSD, Q2 NPN, Q3 NPN, Q4 Q_Dual_NPN_NPN_BRT_E1B1C2E2B2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, SW1 SW_Omron_B3FS, SW2 SW_DIP_x02, SW3 SW_DIP_x02, SW4 SW_Omron_B3FS, U1 TLC272, U10 ESP32-WROOM-32D, U2 MCP4728, U3 XL6008, U4 MT3608, U6 AP2112K-3.3, U7 AP2112K-3.3, U8 AP2112K-3.3, U9 CH340C

Commit message: Arreglo_5V_Pantalla
Parts:
- removed the C4 at (150.2, 57.5)
- removed the C8 at (167.9, 48.0)
- removed the D6 at (159.5, 43.8)
- removed the R10 at (162.8, 52.0)
- removed the R11 at (159.6, 52.8)
- removed the R13 at (163.1, 43.8)
- removed the U4 at (155.7, 56.5)
- added C1: 10u, Capacitor_SMD:C_0805_2012Metric, F.Cu at (164.4, 54.9)
- added C3: 0.1u, Capacitor_SMD:C_0805_2012Metric, F.Cu at (164.4, 56.9)
- added C5: 0.1u, Capacitor_SMD:C_0805_2012Metric, F.Cu at (164.3, 47.2)
- added C7: 22u, Capacitor_SMD:C_0805_2012Metric, F.Cu at (187.4, 22.0)
- added D5: LED, LED_SMD:LED_0603_1608Metric, F.Cu at (191.7, 19.1)
- added JP1: SolderJumper_3_Open, Jumper:SolderJumper-3_P1.3mm_Open_RoundedPad1.0x1.5mm, F.Cu at (187.1, 46.1)
- added PANTALLA2: Conn_01x04_Pin, Connector_JST:JST_XH_B4B-XH-A_1x04_P2.50mm_Vertical, F.Cu at (194.4, 51.2)
- added R3: 54.9k, Resistor_SMD:R_0603_1608Metric, F.Cu at (173.5, 52.8)
- added R6: 10k, Resistor_SMD:R_0603_1608Metric, F.Cu at (173.5, 54.2)
- added R7: 470, Resistor_SMD:R_0603_1608Metric, F.Cu at (173.5, 55.7)
- added R8: 470, Resistor_SMD:R_0603_1608Metric, F.Cu at (187.3, 19.1)
- added U2: TPS562200, Package_TO_SOT_SMD:SOT-23-6, F.Cu at (164.4, 51.3)
- D4: value D_Schottky -> LED; footprint Diode_SMD:D_SMA -> LED_SMD:LED_0603_1608Metric
- L2: value 22u -> 4.7u
- moved 5V1 37.1 mm to (197.1, 23.4), turned to 0 degrees
- moved F3 7.46 mm to (189.7, 59.2)
- moved SW3 7.46 mm to (194.8, 59.2)
- moved D4 7.26 mm to (173.4, 57.2), turned to 180 degrees
- moved Alimentacion_12V1 6.06 mm to (194.9, 68.2)
- moved C2 4.94 mm to (182.3, 63.9)
- moved C21 1.96 mm to (182.0, 42.2), turned to 180 degrees
- moved L2 1.62 mm to (173.8, 46.9), turned to 0 degrees
- renumbered Alimentacion_12V2 to Alimentacion_12V1, C11 to C10, C12 to C11, C13 to C12, C7 to C13, C5 to C14, C14 to C15, C10 to C16, C6 to C17, C15 to C18, C16 to C19, C1 to C2, C17 to C20, C18 to C21, C19 to C22, C20 to C23, C22 to C24, C23 to C25, C2 to C4, C3 to C6, C21 to C8, D5 to D2, D2 to D3, D7 to D6, D8 to D7, D9 to D8, D3 to D9, F2 to F1, F1 to F2, GND2 to GND1, J10 to J1, Q4 to Q2, Q2 to Q3, Q3 to Q4, R6 to R1, R16 to R10, R17 to R11, R7 to R12, R8 to R13, R19 to R14, R20 to R15, R21 to R16, R22 to R17, R23 to R18, R24 to R19, R25 to R20, R18 to R21, R1 to R22, R14 to R23, R26 to R24, R4 to R25, R9 to R26, R3 to R4, R15 to R9, SW2 to SW1, SW3 to SW2, SW6 to SW3, SW1 to SW4, SW4 to SW5, U3 to U1, U6 to U3, U2 to U4, U7 to U5, U8 to U6, U9 to U7, U10 to U8, U1 to U9
Connections:
- D2 pad 1: V+ -> +5V
- D2 pad 2: V_in -> 5DC
- D4 pad 1: +5V -> GND
- D4 pad 2: /SW_5V -> Net-(D4-A)
- L2 pad 1: V+ -> Net-(U2-SW)
- L2 pad 2: /SW_5V -> 5DC
- Q1 pad 1: V_in -> 5DC
- Q1 pad 2: V+ -> +5V
- R1 pad 1: V_in -> 5DC
Routing:
- net +3.3V: track 126.3 -> 222.0 mm, vias 0 -> 1
- net V+: track 66.9 -> 0.00 mm, vias 3 -> 0
- net +5V: track 116.2 -> 169.4 mm, vias 2 -> 4
- net 5DC: track 0.00 -> 46.6 mm, vias 0 -> 2
- net sda: track 91.1 -> 130.8 mm
- net scl: track 111.8 -> 147.5 mm
- net /SW_5V: track 22.0 -> 0.00 mm
- net V_in: track 94.6 -> 73.6 mm
- net Net-(U2-SW): track 0.00 -> 19.4 mm
- net /FB_5V: track 8.05 -> 0.00 mm
- net Net-(JP1-C): track 0.00 -> 7.30 mm
- net Net-(U2-VFB): track 0.00 -> 7.27 mm
- net Net-(U2-VBST): track 0.00 -> 5.76 mm
- net /RESET: track 62.0 -> 66.9 mm
- net Net-(D4-A): track 0.00 -> 3.74 mm
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Other:
- board text added: "3V3"
- board text added: "5V"
- board text added: "SCL SDA V+ GND"
- board text added: "Transiluminador V1.1 Amaru Rubilar 8-2024"
- board text removed: "Transiluminador V1.1 Amaru Rubilar 1-2024"

Commit message: sensor_temp
Parts:
- added J2: Conn_01x02_Pin, Connector_JST:JST_XH_B2B-XH-A_1x02_P2.50mm_Vertical, F.Cu at (113.6, 26.4)
- added R27: 10k, Resistor_SMD:R_0603_1608Metric, F.Cu at (120.7, 24.7)
- moved 3.3V1 14.0 mm to (128.4, 29.1)
- moved VDL1 11.5 mm to (128.4, 34.9)
- moved VS1 10.6 mm to (128.4, 42.0)
- moved R9 7.04 mm to (124.4, 31.6)
- moved C10 6.74 mm to (122.9, 31.6)
- moved U3 6.74 mm to (119.6, 31.8)
- moved C9 6.74 mm to (114.5, 32.4)
- moved C22 4.74 mm to (134.7, 26.9)
- moved R10 3.97 mm to (124.3, 38.5)
- moved C12 3.40 mm to (122.8, 38.5)
- moved U5 3.40 mm to (119.5, 38.7)
- moved C11 3.40 mm to (114.5, 39.9)
- moved D8 3.31 mm to (125.8, 45.0), turned to -90 degrees
- moved D6 3.29 mm to (125.8, 31.6), turned to -90 degrees
- moved C23 3.22 mm to (136.4, 27.0)
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Connections:
- U8 pad 7: unconnected-(U8-IO35-Pad7) -> Temp
Routing:
- net Temp: track 0.00 -> 35.3 mm, vias 0 -> 2
- net GND: track 43.6 -> 63.0 mm, vias 41 -> 42
- net VS_3V3: track 106.1 -> 124.2 mm, vias 3 -> 4
- net VDL_3V3: track 118.3 -> 110.8 mm
- net +5V: track 169.4 -> 162.8 mm
- net Net-(D6-A): track 1.89 -> 3.27 mm
- net Net-(D7-A): track 1.77 -> 2.98 mm
- net Net-(D8-A): track 2.70 -> 3.47 mm
- net UP: track 35.2 -> 34.6 mm

Commit message: Esquematico_LEDS_Test
Parts:
- added Dac1: DAC1, TestPoint:TestPoint_Loop_D2.50mm_Drill1.0mm_LowProfile, F.Cu at (143.0, 65.2)
- added Dac2: DAC2, TestPoint:TestPoint_Loop_D2.50mm_Drill1.0mm_LowProfile, F.Cu at (143.1, 69.3)
Routing:
- net DC: track 60.0 -> 60.8 mm
- net Vdac2: track 17.1 -> 16.4 mm
- net Vdac1: track 17.6 -> 18.1 mm
