File: electronics/controlador/Transiluminador.kicad_sch (KiCad schematic)
At the start: 92 parts, among them J10 USB_B_Micro, Q1 Q_PMOS_GSD, Q2 NPN, Q3 NPN, Q4 Q_Dual_NPN_NPN_BRT_E1B1C2E2B2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, SW1 SW_Omron_B3FS, SW2 SW_DIP_x02, SW3 SW_DIP_x02, SW4 SW_Omron_B3FS, U1 TLC272, U10 ESP32-WROOM-32D, U2 MCP4728, U3 XL6008, U4 MT3608, U6 AP2112K-3.3, U7 AP2112K-3.3, U8 AP2112K-3.3, U9 CH340C

Commit message: Arreglo_5V_Pantalla
Parts:
- removed C4: 22u, Capacitor_SMD:C_0805_2012Metric, symbol IoWLabs:C
- removed D4: D_Schottky, Diode_SMD:D_SMA, symbol Device:D_Schottky
- removed R10: 7K5, Resistor_SMD:R_0603_1608Metric, symbol IoWLabs:RES
- removed R11: 1K, Resistor_SMD:R_0603_1608Metric, symbol IoWLabs:RES
- removed U4: MT3608, Package_TO_SOT_SMD:SOT-23-6, symbol Regulator_Switching:MT3608
- added C1: 10u, Capacitor_SMD:C_0805_2012Metric, symbol IoWLabs:C
- added C3, C5: 0.1u, Capacitor_SMD:C_0805_2012Metric, symbol IoWLabs:C
- added D4: LED, LED_SMD:LED_0603_1608Metric, symbol Device:LED
- added JP1: SolderJumper_3_Open, Jumper:SolderJumper-3_P1.3mm_Open_RoundedPad1.0x1.5mm, symbol Jumper:SolderJumper_3_Open
- added PANTALLA2: Conn_01x04_Pin, Connector_JST:JST_XH_B4B-XH-A_1x04_P2.50mm_Vertical, symbol Connector:Conn_01x04_Pin
- added R3: 54.9k, Resistor_SMD:R_0603_1608Metric, symbol IoWLabs:RES
- added R6: 10k, Resistor_SMD:R_0603_1608Metric, symbol IoWLabs:RES
- added R7: 470, Resistor_SMD:R_0603_1608Metric, symbol IoWLabs:RES
- added U2: TPS562200, Package_TO_SOT_SMD:SOT-23-6, symbol Regulator_Switching:TPS562200
- L2: value 22u -> 4.7u
- renumbered Alimentacion_12V2 to Alimentacion_12V1, C11 to C10, C12 to C11, C13 to C12, C7 to C13, C5 to C14, C14 to C15, C10 to C16, C6 to C17, C15 to C18, C16 to C19, C1 to C2, C17 to C20, C18 to C21, C19 to C22, C20 to C23, C22 to C24, C23 to C25, C2 to C4, C3 to C6, C8 to C7, C21 to C8, D5 to D2, D2 to D3, D6 to D5, D7 to D6, D8 to D7, D9 to D8, D3 to D9, F2 to F1, F1 to F2, GND2 to GND1, J10 to J1, Q4 to Q2, Q2 to Q3, Q3 to Q4, R6 to R1, R16 to R10, R17 to R11, R7 to R12, R8 to R13, R19 to R14, R20 to R15, R21 to R16, R22 to R17, R23 to R18, R24 to R19, R25 to R20, R18 to R21, R1 to R22, R14 to R23, R26 to R24, R4 to R25, R9 to R26, R3 to R4, R13 to R8, R15 to R9, SW2 to SW1, SW3 to SW2, SW6 to SW3, SW1 to SW4, SW4 to SW5, U3 to U1, U6 to U3, U2 to U4, U7 to U5, U8 to U6, U9 to U7, U10 to U8, U1 to U9
Connections:
- net +3V3: now also JP1.3 (B)
- net +5V: now also D2.1 (K), Q1.2 (S), JP1.1 (A)
- net GND: now also C1.2, C3.2, D4.1 (K), PANTALLA2.4 (Pin_4), R6.2, U2.1 (GND)
- net V_in: now also C1.1, C3.1, U2.3 (VIN), U2.5 (EN); no longer D2.2 (A), Q1.1 (G), R1.1
- net scl: now also PANTALLA2.1 (Pin_1)
- net sda: now also PANTALLA2.2 (Pin_2)
- net SW_5V renamed 5DC
- net 5DC: now also D2.2 (A), Q1.1 (G), R1.1, R3.2, R6.1, R7.1
- removed net V+: D2.1 (K), L2.1, Q1.2 (S)
- new net: C5.1, U2.6 (VBST)
- new net: C5.2, L2.1, U2.2 (SW)
- new net: D4.2 (A), R7.2
- new net: R3.1, U2.4 (VFB)
- new net: JP1.2 (C), PANTALLA2.3 (Pin_3)
Other:
- note added: "Pantalla Reemplazo"
- note added: "V_out = 0.765(R20/R21 + 1)"
- note removed: "V_out = 0.6(R8/R7 + 1)"
- moved on the sheet: 5V1, C7, D5, R8

Commit message: sensor_temp
Parts:
- added J2: Conn_01x02_Pin, Connector_JST:JST_XH_B2B-XH-A_1x02_P2.50mm_Vertical, symbol Connector:Conn_01x02_Pin
- added R27: 10k, Resistor_SMD:R_0603_1608Metric, symbol IoWLabs:RES
Connections:
- net GND: now also R27.2
- net VS_3V3: now also J2.1 (Pin_1)
- net Temp: now reaches U8.7 (IO35)
- net Temp: now also J2.2 (Pin_2), R27.1
Other:
- note added: "Sensor de Temperatura"

Commit message: Esquematico_LEDS_Test
Parts:
- added Dac1: DAC1, TestPoint:TestPoint_Loop_D2.50mm_Drill1.0mm_LowProfile, symbol Connector:Conn_01x01_Pin
- added Dac2: DAC2, TestPoint:TestPoint_Loop_D2.50mm_Drill1.0mm_LowProfile, symbol Connector:Conn_01x01_Pin
Connections:
- net Vdac1: now also Dac1.1 (Pin_1)
- net Vdac2: now also Dac2.1 (Pin_1)
Changed lines of the file:
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@@
 	(wire
 		(pts
+			(xy 220.98 59.436) (xy 222.504 59.436)
+		)
+		(stroke
+			(width 0)
+			(type default)
+		)
+	)
+	(wire
+		(pts
 			(xy 273.685 153.035) (xy 273.685 155.575)
 		)
@@
 	(wire
 		(pts
+			(xy 221.234 54.864) (xy 222.504 54.864)
+		)
+		(stroke
+			(width 0)
+			(type default)
+		)
+	)
+	(wire
+		(pts
 			(xy 147.32 153.035) (xy 146.685 153.035)
 		)
@@
 		)
 	)
+	(global_label "Vdac2"
+		(shape input)
+		(at 220.98 59.436 180)
+		(fields_autoplaced yes)
+		(effects
+			(font
+				(size 1.27 1.27)
+			)
+			(justify right)
+		)
+		(property "Intersheetrefs" "${INTERSHEET_REFS}"
+			(at 212.3101 59.436 0)
+			(effects
+				(font
+					(size 1.27 1.27)
+				)
+				(justify right)
+				(hide yes)
+			)
+		)
+	)
 	(global_label "VS_3V3"
 		(shape input)
@@
 		)
 	)
+	(global_label "Vdac1"
+		(shape input)
+		(at 221.234 54.864 180)
+		(fields_autoplaced yes)
+		(effects
+			(font
+				(size 1.27 1.27)
+			)
+			(justify right)
+		)
+		(property "Intersheetrefs" "${INTERSHEET_REFS}"
+			(at 212.5641 54.864 0)
+			(effects
+				(font
+					(size 1.27 1.27)
+				)
+				(justify right)
+				(hide yes)
+			)
+		)
+	)
 	(global_label "VS_3V3"
 		(shape input)
@@
 	)
 	(symbol
+		(lib_id "Connector:Conn_01x01_Pin")
+		(at 227.584 54.864 180)
+		(unit 1)
+		(exclude_from_sim no)
+		(in_bom yes)
+		(on_board yes)
+		(dnp no)
+		(fields_autoplaced yes)
+		(property "Reference" "Dac1"
+			(at 226.949 49.784 0)
+			(effects
+				(font
+					(size 1.27 1.27)
+				)
+			)
+		)
+		(property "Value" "DAC1"
+			(at 226.949 52.324 0)
+			(effects
+				(font
+					(size 1.27 1.27)
+				)
+			)
+		)
+		(property "Footprint" "TestPoint:TestPoint_Loop_D2.50mm_Drill1.0mm_LowProfile"
+			(at 227.584 54.864 0)
+			(effects
+				(font
+					(size 1.27 1.27)
+				)
+				(hide yes)
+			)
+		)
+		(property "Datasheet" "~"
+			(at 227.584 54.864 0)
+			(effects
+				(font
+					(size 1.27 1.27)
+				)
+				(hide yes)
+			)
+		)
+		(property "Description" ""
+			(at 227.584 54.864 0)
+			(effects
+				(font
+					(size 1.27 1.27)
+				)
+				(hide yes)
+			)
+		)
+		(pin "1"
+		)
+		(instances
+			(project "Transiluminador"
+				(path "/3bccb558-cfc1-47b0-87de-a688fdd981c6"
+					(reference "Dac1")
+					(unit 1)
+				)
+			)
+		)
+	)
+	(symbol
 		(lib_id "IoWLabs:RES")
 		(at 273.05 34.925 270)
@@
 					(unit 1)
 				)
+			)
+		)
+	)
+	(symbol
+		(lib_id "Connector:Conn_01x01_Pin")
+		(at 227.584 59.436 180)
+		(unit 1)
+		(exclude_from_sim no)
+		(in_bom yes)
+		(on_board yes)
+		(dnp no)
+		(property "Reference" "Dac2"
+			(at 227.584 57.912 0)
+			(effects
+				(font
+					(size 1.27 1.27)
+				)
+			)
+		)
+		(property "Value" "DAC2"
+			(at 227.584 61.595 0)
+			(effects
+				(font
+					(size 1.27 1.27)
+				)
+			)
+		)
+		(property "Footprint" "TestPoint:TestPoint_Loop_D2.50mm_Drill1.0mm_LowProfile"
+			(at 227.584 59.436 0)
+			(effects
+				(font
+					(size 1.27 1.27)
+				)
+				(hide yes)
+			)
+		)
+		(property "Datasheet" "~"
+			(at 227.584 59.436 0)
+			(effects
+				(font
+					(size 1.27 1.27)
+				)
+				(hide yes)
+			)
+		)
+		(property "Description" ""
+			(at 227.584 59.436 0)
+			(effects
+				(font
+					(size 1.27 1.27)
+				)
+				(hide yes)
+			)
+		)
+		(pin "1"
+		)
+		(instances
+			(project "Transiluminador"
+				(path "/3bccb558-cfc1-47b0-87de-a688fdd981c6"
+					(reference "Dac2")
+					(unit 1)
+				)
