File: electronics/LEDs/LEDs_test/LEDs_test.kicad_pcb (KiCad board)
At the start: 2 copper layers, 73 x 80 mm, 40 parts

Commit message: Letras_PCB
Parts:
- added G***: LOGO, IoWLabsLogos:OpenHardware_10mm, F.Cu at (151.0, 69.0)
- added G***: LOGO, IoWLabsLogos:IoWLabs_logo_13mm, F.Cu at (118.6, 29.9)
- added G***: LOGO, Imagenes_png:Light_Glyph, B.Cu at (128.8, 64.0)
Other:
- board text added: "PCB LEDs de Prueba Amaru Rubilar 08-2024 IoWLabs"
- board text added: "V I GND"
